File: PCB/WindSplit.kicad_sch (KiCad schematic)
At the start: 138 parts, among them SW1 SW_Push_45deg, SW10 SW_Push_45deg, SW11 SW_Push_45deg, SW12 SW_Push_45deg, SW13 SW_Push_45deg, SW14 SW_Push_45deg, SW15 SW_Push_45deg, SW16 SW_Push_45deg, SW17 SW_Push_45deg, SW18 SW_Push_45deg, SW19 SW_Push_45deg, SW2 SW_Push_45deg, SW20 SW_Push_45deg, SW21 SW_Push_45deg, SW22 SW_Push_45deg, SW23 SW_Push_45deg, SW24 SW_Push_45deg, SW25 SW_Push_45deg, SW26 SW_Push_45deg, SW27 SW_Push_45deg, SW28 SW_Push_45deg, SW29 SW_Push_45deg, SW3 SW_Push_45deg, SW30 SW_Push_45deg, SW31 SW_Push_45deg, SW32 SW_Push_45deg, SW33 SW_Push_45deg, SW34 SW_Push_45deg, SW35 SW_Push_45deg, SW36 SW_Push_45deg, SW37 SW_Push_45deg, SW38 SW_Push_45deg, SW39 SW_Push_45deg, SW4 SW_Push_45deg, SW40 SW_Push_45deg, SW41 SW_Push_45deg, SW42 SW_Push_45deg, SW43 SW_Push_45deg, SW44 SW_Push_45deg, SW45 SW_Push_45deg, SW46 SW_Push_45deg, SW47 SW_Push_45deg, SW48 SW_Push_45deg, SW49 SW_Push_45deg, SW5 SW_Push_45deg, SW50 SW_Push_45deg, SW51 SW_Push_45deg, SW52 SW_Push_45deg, SW53 SW_Push_45deg, SW54 SW_Push_45deg, SW55 SW_Push_45deg, SW56 SW_Push_45deg, SW57 SW_Push_45deg, SW58 SW_Push_45deg, SW59 SW_Push_45deg, SW6 SW_Push_45deg, SW60 SW_Push_45deg, SW61 SW_Push_45deg, SW62 SW_Push_45deg, SW63 SW_Push_45deg, SW64 SW_Push_45deg, SW65 SW_Push_45deg, SW66 SW_Push_45deg, SW67 SW_Push_45deg, SW68 SW_Push_45deg, SW7 SW_Push_45deg, SW8 SW_Push_45deg, SW9 SW_Push_45deg, U1 Nice_Nano_V2, U2 MCP23017_SP

Commit message: added silk screen
Connections:
- net COL15 is gone; now on net COL14: SW15.1, SW30.1, SW44.1, SW58.1, SW68.1, U2.27 (GPA6)
- net COL1: now also SW17.1, SW2.1, SW32.1, SW46.1, SW60.1, U2.2 (GPB1); no longer SW1.1, SW16.1, SW31.1, SW45.1, SW59.1, U2.1 (GPB0)
- net COL10: now also SW11.1, SW26.1, SW41.1, SW55.1, SW65.1, U2.23 (GPA2); no longer SW10.1, SW25.1, SW40.1, SW54.1, SW64.1, U2.22 (GPA1)
- net COL11: now also SW12.1, SW27.1, SW42.1, SW56.1, SW66.1, U2.24 (GPA3); no longer SW11.1, SW26.1, SW41.1, SW55.1, SW65.1, U2.23 (GPA2)
- net COL12: now also SW13.1, SW28.1, U2.25 (GPA4); no longer SW12.1, SW27.1, SW42.1, SW56.1, SW66.1, U2.24 (GPA3)
- net COL13: now also SW14.1, SW29.1, SW43.1, SW57.1, SW67.1, U2.26 (GPA5); no longer SW13.1, SW28.1, U2.25 (GPA4)
- net COL14: no longer SW14.1, SW29.1, SW43.1, SW57.1, SW67.1, U2.26 (GPA5)
- net COL2: now also SW18.1, SW3.1, SW33.1, SW47.1, SW61.1, U2.3 (GPB2); no longer SW17.1, SW2.1, SW32.1, SW46.1, SW60.1, U2.2 (GPB1)
- net COL3: now also SW19.1, SW34.1, SW4.1, SW48.1, U2.4 (GPB3); no longer SW18.1, SW3.1, SW33.1, SW47.1, SW61.1, U2.3 (GPB2)
- net COL4: now also SW20.1, SW35.1, SW49.1, SW5.1, U2.5 (GPB4); no longer SW19.1, SW34.1, SW4.1, SW48.1, U2.4 (GPB3)
- net COL5: now also SW21.1, SW36.1, SW50.1, SW6.1, SW62.1, U2.6 (GPB5); no longer SW20.1, SW35.1, SW49.1, SW5.1, U2.5 (GPB4)
- net COL6: now also SW22.1, SW37.1, SW51.1, SW7.1, U2.7 (GPB6); no longer SW21.1, SW36.1, SW50.1, SW6.1, SW62.1, U2.6 (GPB5)
- net COL7: now also SW23.1, SW38.1, SW52.1, SW8.1, U2.8 (GPB7); no longer SW22.1, SW37.1, SW51.1, SW7.1, U2.7 (GPB6)
- net COL8: now also SW24.1, SW39.1, SW53.1, SW63.1, SW9.1, U2.21 (GPA0); no longer SW23.1, SW38.1, SW52.1, SW8.1, U2.8 (GPB7)
- net COL9: now also SW10.1, SW25.1, SW40.1, SW54.1, SW64.1, U2.22 (GPA1); no longer SW24.1, SW39.1, SW53.1, SW63.1, SW9.1, U2.21 (GPA0)
- new net COL0: SW1.1, SW16.1, SW31.1, SW45.1, SW59.1, U2.1 (GPB0)
