File: PCB/wind75.kicad_sch (KiCad schematic)
At the start: 138 parts, among them SW1 SW_Push_45deg, SW10 SW_Push_45deg, SW11 SW_Push_45deg, SW12 SW_Push_45deg, SW13 SW_Push_45deg, SW14 SW_Push_45deg, SW15 SW_Push_45deg, SW16 SW_Push_45deg, SW17 SW_Push_45deg, SW18 SW_Push_45deg, SW19 SW_Push_45deg, SW2 SW_Push_45deg, SW20 SW_Push_45deg, SW21 SW_Push_45deg, SW22 SW_Push_45deg, SW23 SW_Push_45deg, SW24 SW_Push_45deg, SW25 SW_Push_45deg, SW26 SW_Push_45deg, SW27 SW_Push_45deg, SW28 SW_Push_45deg, SW29 SW_Push_45deg, SW3 SW_Push_45deg, SW30 SW_Push_45deg, SW31 SW_Push_45deg, SW32 SW_Push_45deg, SW33 SW_Push_45deg, SW34 SW_Push_45deg, SW35 SW_Push_45deg, SW36 SW_Push_45deg, SW37 SW_Push_45deg, SW38 SW_Push_45deg, SW39 SW_Push_45deg, SW4 SW_Push_45deg, SW40 SW_Push_45deg, SW41 SW_Push_45deg, SW42 SW_Push_45deg, SW43 SW_Push_45deg, SW44 SW_Push_45deg, SW45 SW_Push_45deg, SW46 SW_Push_45deg, SW47 SW_Push_45deg, SW48 SW_Push_45deg, SW49 SW_Push_45deg, SW5 SW_Push_45deg, SW50 SW_Push_45deg, SW51 SW_Push_45deg, SW52 SW_Push_45deg, SW53 SW_Push_45deg, SW54 SW_Push_45deg, SW55 SW_Push_45deg, SW56 SW_Push_45deg, SW57 SW_Push_45deg, SW58 SW_Push_45deg, SW59 SW_Push_45deg, SW6 SW_Push_45deg, SW60 SW_Push_45deg, SW61 SW_Push_45deg, SW62 SW_Push_45deg, SW63 SW_Push_45deg, SW64 SW_Push_45deg, SW65 SW_Push_45deg, SW66 SW_Push_45deg, SW67 SW_Push_45deg, SW68 SW_Push_45deg, SW7 SW_Push_45deg, SW8 SW_Push_45deg, SW9 SW_Push_45deg, U1 Nice_Nano_V2, U2 MCP23017_SP

Commit message: review (not finished)
Parts:
- added D1, D10, D11, D12, D13, D14, D15, D2, D3, D4, D5, D58, D6, D7, D8, D9: D, ScottoKeebs_Components:Diode_SOD-123, symbol Device:D
- added SW1, SW10, SW11, SW12, SW13, SW14, SW15, SW2, SW3, SW4, SW5, SW58, SW6, SW7, SW8, SW9: SW_Push_45deg, ScottoKeebs_Hotswap:Hotswap_MX_1.00u, symbol Switch:SW_Push_45deg
- D16: renamed from D1; footprint Diode_THT:D_DO-35_SOD27_P7.62mm_Horizontal -> ScottoKeebs_Components:Diode_SOD-123
- D17: renamed from D2; footprint Diode_THT:D_DO-35_SOD27_P7.62mm_Horizontal -> ScottoKeebs_Components:Diode_SOD-123
- D18: renamed from D3; footprint Diode_THT:D_DO-35_SOD27_P7.62mm_Horizontal -> ScottoKeebs_Components:Diode_SOD-123
- D19: renamed from D4; footprint Diode_THT:D_DO-35_SOD27_P7.62mm_Horizontal -> ScottoKeebs_Components:Diode_SOD-123
- D20: renamed from D5; footprint Diode_THT:D_DO-35_SOD27_P7.62mm_Horizontal -> ScottoKeebs_Components:Diode_SOD-123
- D21: renamed from D6; footprint Diode_THT:D_DO-35_SOD27_P7.62mm_Horizontal -> ScottoKeebs_Components:Diode_SOD-123
- D22: renamed from D7; footprint Diode_THT:D_DO-35_SOD27_P7.62mm_Horizontal -> ScottoKeebs_Components:Diode_SOD-123
- D23: renamed from D8; footprint Diode_THT:D_DO-35_SOD27_P7.62mm_Horizontal -> ScottoKeebs_Components:Diode_SOD-123
- D24: renamed from D9; footprint Diode_THT:D_DO-35_SOD27_P7.62mm_Horizontal -> ScottoKeebs_Components:Diode_SOD-123
- D25: renamed from D10; footprint Diode_THT:D_DO-35_SOD27_P7.62mm_Horizontal -> ScottoKeebs_Components:Diode_SOD-123
- D26: renamed from D11; footprint Diode_THT:D_DO-35_SOD27_P7.62mm_Horizontal -> ScottoKeebs_Components:Diode_SOD-123
- D27: renamed from D12; footprint Diode_THT:D_DO-35_SOD27_P7.62mm_Horizontal -> ScottoKeebs_Components:Diode_SOD-123
- D28: renamed from D13; footprint Diode_THT:D_DO-35_SOD27_P7.62mm_Horizontal -> ScottoKeebs_Components:Diode_SOD-123
- D29: renamed from D14; footprint Diode_THT:D_DO-35_SOD27_P7.62mm_Horizontal -> ScottoKeebs_Components:Diode_SOD-123
- D30: renamed from D15; footprint Diode_THT:D_DO-35_SOD27_P7.62mm_Horizontal -> ScottoKeebs_Components:Diode_SOD-123
- D31: renamed from D16; footprint Diode_THT:D_DO-35_SOD27_P7.62mm_Horizontal -> ScottoKeebs_Components:Diode_SOD-123
- D32: renamed from D17; footprint Diode_THT:D_DO-35_SOD27_P7.62mm_Horizontal -> ScottoKeebs_Components:Diode_SOD-123
- D33: renamed from D18; footprint Diode_THT:D_DO-35_SOD27_P7.62mm_Horizontal -> ScottoKeebs_Components:Diode_SOD-123
- D34: renamed from D19; footprint Diode_THT:D_DO-35_SOD27_P7.62mm_Horizontal -> ScottoKeebs_Components:Diode_SOD-123
- D35: renamed from D20; footprint Diode_THT:D_DO-35_SOD27_P7.62mm_Horizontal -> ScottoKeebs_Components:Diode_SOD-123
- D36: renamed from D21; footprint Diode_THT:D_DO-35_SOD27_P7.62mm_Horizontal -> ScottoKeebs_Components:Diode_SOD-123
- D37: renamed from D22; footprint Diode_THT:D_DO-35_SOD27_P7.62mm_Horizontal -> ScottoKeebs_Components:Diode_SOD-123
- D38: renamed from D23; footprint Diode_THT:D_DO-35_SOD27_P7.62mm_Horizontal -> ScottoKeebs_Components:Diode_SOD-123
- D39: renamed from D24; footprint Diode_THT:D_DO-35_SOD27_P7.62mm_Horizontal -> ScottoKeebs_Components:Diode_SOD-123
- D40: renamed from D25; footprint Diode_THT:D_DO-35_SOD27_P7.62mm_Horizontal -> ScottoKeebs_Components:Diode_SOD-123
- D41: renamed from D26; footprint Diode_THT:D_DO-35_SOD27_P7.62mm_Horizontal -> ScottoKeebs_Components:Diode_SOD-123
- D42: renamed from D27; footprint Diode_THT:D_DO-35_SOD27_P7.62mm_Horizontal -> ScottoKeebs_Components:Diode_SOD-123
- D43: renamed from D28; footprint Diode_THT:D_DO-35_SOD27_P7.62mm_Horizontal -> ScottoKeebs_Components:Diode_SOD-123
- D44: renamed from D29; footprint Diode_THT:D_DO-35_SOD27_P7.62mm_Horizontal -> ScottoKeebs_Components:Diode_SOD-123
- D45: renamed from D30; footprint Diode_THT:D_DO-35_SOD27_P7.62mm_Horizontal -> ScottoKeebs_Components:Diode_SOD-123
- D46: renamed from D31; footprint Diode_THT:D_DO-35_SOD27_P7.62mm_Horizontal -> ScottoKeebs_Components:Diode_SOD-123
- D47: renamed from D32; footprint Diode_THT:D_DO-35_SOD27_P7.62mm_Horizontal -> ScottoKeebs_Components:Diode_SOD-123
- D48: renamed from D33; footprint Diode_THT:D_DO-35_SOD27_P7.62mm_Horizontal -> ScottoKeebs_Components:Diode_SOD-123
- D49: renamed from D34; footprint Diode_THT:D_DO-35_SOD27_P7.62mm_Horizontal -> ScottoKeebs_Components:Diode_SOD-123
- D50: renamed from D35; footprint Diode_THT:D_DO-35_SOD27_P7.62mm_Horizontal -> ScottoKeebs_Components:Diode_SOD-123
- D51: renamed from D36; footprint Diode_THT:D_DO-35_SOD27_P7.62mm_Horizontal -> ScottoKeebs_Components:Diode_SOD-123
- D52: renamed from D37; footprint Diode_THT:D_DO-35_SOD27_P7.62mm_Horizontal -> ScottoKeebs_Components:Diode_SOD-123
- D53: renamed from D38; footprint Diode_THT:D_DO-35_SOD27_P7.62mm_Horizontal -> ScottoKeebs_Components:Diode_SOD-123
- D54: renamed from D39; footprint Diode_THT:D_DO-35_SOD27_P7.62mm_Horizontal -> ScottoKeebs_Components:Diode_SOD-123
- D55: renamed from D40; footprint Diode_THT:D_DO-35_SOD27_P7.62mm_Horizontal -> ScottoKeebs_Components:Diode_SOD-123
- D56: renamed from D41; footprint Diode_THT:D_DO-35_SOD27_P7.62mm_Horizontal -> ScottoKeebs_Components:Diode_SOD-123
- D57: renamed from D42; footprint Diode_THT:D_DO-35_SOD27_P7.62mm_Horizontal -> ScottoKeebs_Components:Diode_SOD-123
- D59: renamed from D43; footprint Diode_THT:D_DO-35_SOD27_P7.62mm_Horizontal -> ScottoKeebs_Components:Diode_SOD-123
- D60: renamed from D44; footprint Diode_THT:D_DO-35_SOD27_P7.62mm_Horizontal -> ScottoKeebs_Components:Diode_SOD-123
- D61: renamed from D45; footprint Diode_THT:D_DO-35_SOD27_P7.62mm_Horizontal -> ScottoKeebs_Components:Diode_SOD-123
- D62: renamed from D46; footprint Diode_THT:D_DO-35_SOD27_P7.62mm_Horizontal -> ScottoKeebs_Components:Diode_SOD-123
- D63: renamed from D47; footprint Diode_THT:D_DO-35_SOD27_P7.62mm_Horizontal -> ScottoKeebs_Components:Diode_SOD-123
- D64: renamed from D48; footprint Diode_THT:D_DO-35_SOD27_P7.62mm_Horizontal -> ScottoKeebs_Components:Diode_SOD-123
- D65: renamed from D49; footprint Diode_THT:D_DO-35_SOD27_P7.62mm_Horizontal -> ScottoKeebs_Components:Diode_SOD-123
- D66: renamed from D50; footprint Diode_THT:D_DO-35_SOD27_P7.62mm_Horizontal -> ScottoKeebs_Components:Diode_SOD-123
- D67: renamed from D51; footprint Diode_THT:D_DO-35_SOD27_P7.62mm_Horizontal -> ScottoKeebs_Components:Diode_SOD-123
- D68: renamed from D52; footprint Diode_THT:D_DO-35_SOD27_P7.62mm_Horizontal -> ScottoKeebs_Components:Diode_SOD-123
- D69: renamed from D53; footprint Diode_THT:D_DO-35_SOD27_P7.62mm_Horizontal -> ScottoKeebs_Components:Diode_SOD-123
- D70: renamed from D54; footprint Diode_THT:D_DO-35_SOD27_P7.62mm_Horizontal -> ScottoKeebs_Components:Diode_SOD-123
- D71: renamed from D55; footprint Diode_THT:D_DO-35_SOD27_P7.62mm_Horizontal -> ScottoKeebs_Components:Diode_SOD-123
- D72: renamed from D56; footprint Diode_THT:D_DO-35_SOD27_P7.62mm_Horizontal -> ScottoKeebs_Components:Diode_SOD-123
- D73: renamed from D57; footprint Diode_THT:D_DO-35_SOD27_P7.62mm_Horizontal -> ScottoKeebs_Components:Diode_SOD-123
- D74: renamed from D58; footprint Diode_THT:D_DO-35_SOD27_P7.62mm_Horizontal -> ScottoKeebs_Components:Diode_SOD-123
- D75: renamed from D59; footprint Diode_THT:D_DO-35_SOD27_P7.62mm_Horizontal -> ScottoKeebs_Components:Diode_SOD-123
- D76: renamed from D60; footprint Diode_THT:D_DO-35_SOD27_P7.62mm_Horizontal -> ScottoKeebs_Components:Diode_SOD-123
- D77: renamed from D61; footprint Diode_THT:D_DO-35_SOD27_P7.62mm_Horizontal -> ScottoKeebs_Components:Diode_SOD-123
- D78: renamed from D62; footprint Diode_THT:D_DO-35_SOD27_P7.62mm_Horizontal -> ScottoKeebs_Components:Diode_SOD-123
- D79: renamed from D63; footprint Diode_THT:D_DO-35_SOD27_P7.62mm_Horizontal -> ScottoKeebs_Components:Diode_SOD-123
- D80: renamed from D64; footprint Diode_THT:D_DO-35_SOD27_P7.62mm_Horizontal -> ScottoKeebs_Components:Diode_SOD-123
- D81: renamed from D65; footprint Diode_THT:D_DO-35_SOD27_P7.62mm_Horizontal -> ScottoKeebs_Components:Diode_SOD-123
- D82: renamed from D66; footprint Diode_THT:D_DO-35_SOD27_P7.62mm_Horizontal -> ScottoKeebs_Components:Diode_SOD-123
- D83: renamed from D67; footprint Diode_THT:D_DO-35_SOD27_P7.62mm_Horizontal -> ScottoKeebs_Components:Diode_SOD-123
- D84: renamed from D68; footprint Diode_THT:D_DO-35_SOD27_P7.62mm_Horizontal -> ScottoKeebs_Components:Diode_SOD-123
- SW16: renamed from SW1; footprint ScottoKeebs_Scotto:MX_Hotswap_1.00u -> ScottoKeebs_Hotswap:Hotswap_MX_1.00u
- SW17: renamed from SW2; footprint ScottoKeebs_Scotto:MX_Hotswap_1.00u -> ScottoKeebs_Hotswap:Hotswap_MX_1.00u
- SW18: renamed from SW3; footprint ScottoKeebs_Scotto:MX_Hotswap_1.00u -> ScottoKeebs_Hotswap:Hotswap_MX_1.00u
- SW19: renamed from SW4; footprint ScottoKeebs_Scotto:MX_Hotswap_1.00u -> ScottoKeebs_Hotswap:Hotswap_MX_1.00u
- SW20: renamed from SW5; footprint ScottoKeebs_Scotto:MX_Hotswap_1.00u -> ScottoKeebs_Hotswap:Hotswap_MX_1.00u
- SW21: renamed from SW6; footprint ScottoKeebs_Scotto:MX_Hotswap_1.00u -> ScottoKeebs_Hotswap:Hotswap_MX_1.00u
- SW22: renamed from SW7; footprint ScottoKeebs_Scotto:MX_Hotswap_1.00u -> ScottoKeebs_Hotswap:Hotswap_MX_1.00u
- SW23: renamed from SW8; footprint ScottoKeebs_Scotto:MX_Hotswap_1.00u -> ScottoKeebs_Hotswap:Hotswap_MX_1.00u
- SW24: renamed from SW9; footprint ScottoKeebs_Scotto:MX_Hotswap_1.00u -> ScottoKeebs_Hotswap:Hotswap_MX_1.00u
- SW25: renamed from SW10; footprint ScottoKeebs_Scotto:MX_Hotswap_1.00u -> ScottoKeebs_Hotswap:Hotswap_MX_1.00u
- SW26: renamed from SW11; footprint ScottoKeebs_Scotto:MX_Hotswap_1.00u -> ScottoKeebs_Hotswap:Hotswap_MX_1.00u
- SW27: renamed from SW12; footprint ScottoKeebs_Scotto:MX_Hotswap_1.00u -> ScottoKeebs_Hotswap:Hotswap_MX_1.00u
- SW28: renamed from SW13; footprint ScottoKeebs_Scotto:MX_Hotswap_1.00u -> ScottoKeebs_Hotswap:Hotswap_MX_1.00u
- SW29: renamed from SW14; footprint ScottoKeebs_Scotto:MX_Hotswap_1.00u -> ScottoKeebs_Hotswap:Hotswap_MX_1.00u
- SW30: renamed from SW15; footprint ScottoKeebs_Scotto:MX_Hotswap_1.00u -> ScottoKeebs_Hotswap:Hotswap_MX_2.00u
- SW31: renamed from SW16; footprint ScottoKeebs_Scotto:MX_Hotswap_1.00u -> ScottoKeebs_Hotswap:Hotswap_MX_1.00u
- SW32: renamed from SW17; footprint ScottoKeebs_Scotto:MX_Hotswap_1.00u -> ScottoKeebs_Hotswap:Hotswap_MX_1.50u
- SW33: renamed from SW18; footprint ScottoKeebs_Scotto:MX_Hotswap_1.00u -> ScottoKeebs_Hotswap:Hotswap_MX_1.00u
- SW34: renamed from SW19; footprint ScottoKeebs_Scotto:MX_Hotswap_1.00u -> ScottoKeebs_Hotswap:Hotswap_MX_1.00u
- SW35: renamed from SW20; footprint ScottoKeebs_Scotto:MX_Hotswap_1.00u -> ScottoKeebs_Hotswap:Hotswap_MX_1.00u
- SW36: renamed from SW21; footprint ScottoKeebs_Scotto:MX_Hotswap_1.00u -> ScottoKeebs_Hotswap:Hotswap_MX_1.00u
- SW37: renamed from SW22; footprint ScottoKeebs_Scotto:MX_Hotswap_1.00u -> ScottoKeebs_Hotswap:Hotswap_MX_1.00u
- SW38: renamed from SW23; footprint ScottoKeebs_Scotto:MX_Hotswap_1.00u -> ScottoKeebs_Hotswap:Hotswap_MX_1.00u
- SW39: renamed from SW24; footprint ScottoKeebs_Scotto:MX_Hotswap_1.00u -> ScottoKeebs_Hotswap:Hotswap_MX_1.00u
- SW40: renamed from SW25; footprint ScottoKeebs_Scotto:MX_Hotswap_1.00u -> ScottoKeebs_Hotswap:Hotswap_MX_1.00u
- SW41: renamed from SW26; footprint ScottoKeebs_Scotto:MX_Hotswap_1.00u -> ScottoKeebs_Hotswap:Hotswap_MX_1.00u
- SW42: renamed from SW27; footprint ScottoKeebs_Scotto:MX_Hotswap_1.00u -> ScottoKeebs_Hotswap:Hotswap_MX_1.00u
- SW43: renamed from SW28; footprint ScottoKeebs_Scotto:MX_Hotswap_1.00u -> ScottoKeebs_Hotswap:Hotswap_MX_1.00u
- SW44: renamed from SW29; footprint ScottoKeebs_Scotto:MX_Hotswap_1.00u -> ScottoKeebs_Hotswap:Hotswap_MX_1.00u
- SW45: renamed from SW30; footprint ScottoKeebs_Scotto:MX_Hotswap_1.00u -> ScottoKeebs_Hotswap:Hotswap_MX_1.50u
- SW46: renamed from SW31; footprint ScottoKeebs_Scotto:MX_Hotswap_1.00u -> ScottoKeebs_Hotswap:Hotswap_MX_1.00u
- SW47: renamed from SW32; footprint ScottoKeebs_Scotto:MX_Hotswap_1.00u -> ScottoKeebs_Hotswap:Hotswap_MX_1.75u
- SW48: renamed from SW33; footprint ScottoKeebs_Scotto:MX_Hotswap_1.00u -> ScottoKeebs_Hotswap:Hotswap_MX_1.00u
- SW49: renamed from SW34; footprint ScottoKeebs_Scotto:MX_Hotswap_1.00u -> ScottoKeebs_Hotswap:Hotswap_MX_1.00u
- SW50: renamed from SW35; footprint ScottoKeebs_Scotto:MX_Hotswap_1.00u -> ScottoKeebs_Hotswap:Hotswap_MX_1.00u
- SW51: renamed from SW36; footprint ScottoKeebs_Scotto:MX_Hotswap_1.00u -> ScottoKeebs_Hotswap:Hotswap_MX_1.00u
- SW52: renamed from SW37; footprint ScottoKeebs_Scotto:MX_Hotswap_1.00u -> ScottoKeebs_Hotswap:Hotswap_MX_1.00u
- SW53: renamed from SW38; footprint ScottoKeebs_Scotto:MX_Hotswap_1.00u -> ScottoKeebs_Hotswap:Hotswap_MX_1.00u
- SW54: renamed from SW39; footprint ScottoKeebs_Scotto:MX_Hotswap_1.00u -> ScottoKeebs_Hotswap:Hotswap_MX_1.00u
- SW55: renamed from SW40; footprint ScottoKeebs_Scotto:MX_Hotswap_1.00u -> ScottoKeebs_Hotswap:Hotswap_MX_1.00u
- SW56: renamed from SW41; footprint ScottoKeebs_Scotto:MX_Hotswap_1.00u -> ScottoKeebs_Hotswap:Hotswap_MX_1.00u
- SW57: renamed from SW42; footprint ScottoKeebs_Scotto:MX_Hotswap_1.00u -> ScottoKeebs_Hotswap:Hotswap_MX_1.00u
- SW59: renamed from SW43; footprint ScottoKeebs_Scotto:MX_Hotswap_1.00u -> ScottoKeebs_Hotswap:Hotswap_MX_2.25u
- SW60: renamed from SW44; footprint ScottoKeebs_Scotto:MX_Hotswap_1.00u -> ScottoKeebs_Hotswap:Hotswap_MX_1.00u
- SW61: renamed from SW45; footprint ScottoKeebs_Scotto:MX_Hotswap_1.00u -> ScottoKeebs_Hotswap:Hotswap_MX_2.25u
- SW62: renamed from SW46; footprint ScottoKeebs_Scotto:MX_Hotswap_1.00u -> ScottoKeebs_Hotswap:Hotswap_MX_1.00u
- SW63: renamed from SW47; footprint ScottoKeebs_Scotto:MX_Hotswap_1.00u -> ScottoKeebs_Hotswap:Hotswap_MX_1.00u
- SW64: renamed from SW48; footprint ScottoKeebs_Scotto:MX_Hotswap_1.00u -> ScottoKeebs_Hotswap:Hotswap_MX_1.00u
- SW65: renamed from SW49; footprint ScottoKeebs_Scotto:MX_Hotswap_1.00u -> ScottoKeebs_Hotswap:Hotswap_MX_1.00u
- SW66: renamed from SW50; footprint ScottoKeebs_Scotto:MX_Hotswap_1.00u -> ScottoKeebs_Hotswap:Hotswap_MX_1.00u
- SW67: renamed from SW51; footprint ScottoKeebs_Scotto:MX_Hotswap_1.00u -> ScottoKeebs_Hotswap:Hotswap_MX_1.00u
- SW68: renamed from SW52; footprint ScottoKeebs_Scotto:MX_Hotswap_1.00u -> ScottoKeebs_Hotswap:Hotswap_MX_1.00u
- SW69: renamed from SW53; footprint ScottoKeebs_Scotto:MX_Hotswap_1.00u -> ScottoKeebs_Hotswap:Hotswap_MX_1.00u
- SW70: renamed from SW54; footprint ScottoKeebs_Scotto:MX_Hotswap_1.00u -> ScottoKeebs_Hotswap:Hotswap_MX_1.00u
- SW71: renamed from SW55; footprint ScottoKeebs_Scotto:MX_Hotswap_1.00u -> ScottoKeebs_Hotswap:Hotswap_MX_1.00u
- SW72: renamed from SW56; footprint ScottoKeebs_Scotto:MX_Hotswap_1.00u -> ScottoKeebs_Hotswap:Hotswap_MX_1.75u
- SW73: renamed from SW57; footprint ScottoKeebs_Scotto:MX_Hotswap_1.00u -> ScottoKeebs_Hotswap:Hotswap_MX_1.00u
- SW74: renamed from SW58; footprint ScottoKeebs_Scotto:MX_Hotswap_1.00u -> ScottoKeebs_Hotswap:Hotswap_MX_1.00u
- SW75: renamed from SW59; footprint ScottoKeebs_Scotto:MX_Hotswap_1.00u -> ScottoKeebs_Hotswap:Hotswap_MX_1.25u
- SW76: renamed from SW60; footprint ScottoKeebs_Scotto:MX_Hotswap_1.00u -> ScottoKeebs_Hotswap:Hotswap_MX_1.25u
- SW77: renamed from SW61; footprint ScottoKeebs_Scotto:MX_Hotswap_1.00u -> ScottoKeebs_Hotswap:Hotswap_MX_1.25u
- SW78: renamed from SW62; footprint ScottoKeebs_Scotto:MX_Hotswap_1.00u -> ScottoKeebs_Hotswap:Hotswap_MX_6.25u
- SW79: renamed from SW63; footprint ScottoKeebs_Scotto:MX_Hotswap_1.00u -> ScottoKeebs_Hotswap:Hotswap_MX_1.00u
- SW80: renamed from SW64; footprint ScottoKeebs_Scotto:MX_Hotswap_1.00u -> ScottoKeebs_Hotswap:Hotswap_MX_1.00u
- SW81: renamed from SW65; footprint ScottoKeebs_Scotto:MX_Hotswap_1.00u -> ScottoKeebs_Hotswap:Hotswap_MX_1.00u
- SW82: renamed from SW66; footprint ScottoKeebs_Scotto:MX_Hotswap_1.00u -> ScottoKeebs_Hotswap:Hotswap_MX_1.00u
- SW83: renamed from SW67; footprint ScottoKeebs_Scotto:MX_Hotswap_1.00u -> ScottoKeebs_Hotswap:Hotswap_MX_1.00u
- SW84: renamed from SW68; footprint ScottoKeebs_Scotto:MX_Hotswap_1.00u -> ScottoKeebs_Hotswap:Hotswap_MX_1.00u
Connections:
- net COL0: now also SW1.1
- net COL1: now also SW2.1
- net COL10: now also SW11.1
- net COL11: now also SW12.1
- net COL12: now also SW13.1, SW58.1
- net COL13: now also SW14.1
- net COL14: now also SW15.1
- net COL2: now also SW3.1
- net COL3: now also SW4.1
- net COL4: now also SW5.1
- net COL5: now also SW6.1
- net COL6: now also SW7.1
- net COL7: now also SW8.1
- net COL8: now also SW9.1
- net COL9: now also SW10.1
- net ROW3: now also D58.1 (K)
- net ROW0: now reaches U1.18 (19)
- net ROW0: now also D1.1 (K), D10.1 (K), D11.1 (K), D12.1 (K), D13.1 (K), D14.1 (K), D15.1 (K), D2.1 (K), D3.1 (K), D4.1 (K), D5.1 (K), D6.1 (K), D7.1 (K), D8.1 (K), D9.1 (K)
- new net: D58.2 (A), SW58.2
- new net: D5.2 (A), SW5.2
- new net: D2.2 (A), SW2.2
- new net: D11.2 (A), SW11.2
- new net: D12.2 (A), SW12.2
- new net: D9.2 (A), SW9.2
- new net: D1.2 (A), SW1.2
- new net: D6.2 (A), SW6.2
- new net: D13.2 (A), SW13.2
- new net: D3.2 (A), SW3.2
- new net: D7.2 (A), SW7.2
- new net: D15.2 (A), SW15.2
- new net: D8.2 (A), SW8.2
- new net: D4.2 (A), SW4.2
- new net: D14.2 (A), SW14.2
- new net: D10.2 (A), SW10.2
